File: battery_ind.sch (KiCad schematic (older format))
At the start: 9 parts, among them U13 LM393

Commit message: Fix battery indicator layout
Parts:
- D3: value ZENER -> ZENER (5.1V); footprint Diodes_SMD:SOD-123 -> trac-2:SOD-123
- R11: value 8k -> 220
- R36: value 10.5k -> 10k
Connections:
- net GND: now also D3.1 (A); no longer D3.2 (K)
- net at R11.1, R7.2: now also D3.2 (K); no longer D3.1 (A)
- net Vin renamed Vbat
Changed lines of the file:
@@
 P 5400 4250
 F 0 "R36" V 5480 4250 40  0000 C CNN
-F 1 "10.5k" V 5407 4251 40  0000 C CNN
+F 1 "10k" V 5407 4251 40  0000 C CNN
 F 2 "Resistors_SMD:R_0805" V 5330 4250 30  0001 C CNN
 F 3 "" H 5400 4250 30  0000 C CNN
@@
 P 5400 3550
 F 0 "R11" V 5480 3550 40  0000 C CNN
-F 1 "8k" V 5407 3551 40  0000 C CNN
+F 1 "220" V 5407 3551 40  0000 C CNN
 F 2 "Resistors_SMD:R_0805" V 5330 3550 30  0001 C CNN
 F 3 "" H 5400 3550 30  0000 C CNN
@@
 Wire Wire Line
 	5400 3300 5400 3100
-$Comp
-L ZENER D3
-U 1 1 56A176AC
-P 5050 3700
-F 0 "D3" H 5050 3800 50  0000 C CNN
-F 1 "ZENER" H 5050 3600 40  0000 C CNN
-F 2 "Diodes_SMD:SOD-123" H 5050 3700 60  0001 C CNN
-F 3 "" H 5050 3700 60  0000 C CNN
-	1    5050 3700
-	0    1    1    0
-$EndComp
 Wire Wire Line
 	5400 3200 5050 3200
@@
 Connection ~ 5400 4500
 Text HLabel 4200 2500 0    60   Input ~ 0
-Vin
+Vbat
 Wire Wire Line
 	4200 2500 6350 2500
@@
 Text Notes 4950 4950 0    60   ~ 0
 Low Battery Voltage Indicator
+$Comp
+L ZENER D3
+U 1 1 56BFDFF8
+P 5050 3700
+F 0 "D3" H 5050 3800 50  0000 C CNN
+F 1 "ZENER (5.1V)" H 5050 3600 40  0000 C CNN
+F 2 "trac-2:SOD-123" H 5050 3700 60  0001 C CNN
+F 3 "" H 5050 3700 60  0000 C CNN
+	1    5050 3700
+	0    -1   -1   0
+$EndComp
 $EndSCHEMATC

Commit message: Clean up labels, fix diode pin numbers, break out remaining open pins on PIC
Parts:
- R38: value 5k -> 4.99k
Changed lines of the file:
@@
 $EndComp
 $Comp
-L GND #PWR022
+L GND #PWR22
 U 1 1 56A16A0B
 P 6350 4650
-F 0 "#PWR022" H 6350 4650 30  0001 C CNN
+F 0 "#PWR22" H 6350 4650 30  0001 C CNN
 F 1 "GND" H 6350 4580 30  0001 C CNN
 F 2 "" H 6350 4650 60  0000 C CNN
@@
 P 5750 4250
 F 0 "R38" V 5830 4250 40  0000 C CNN
-F 1 "5k" V 5757 4251 40  0000 C CNN
+F 1 "4.99k" V 5757 4251 40  0000 C CNN
 F 2 "Resistors_SMD:R_0805" V 5680 4250 30  0001 C CNN
 F 3 "" H 5750 4250 30  0000 C CNN
